Commit message: Moved URDF models into their own folder. Also, added a couple more URDF models.

File: Utilities/URDF_Models/kuka_lwr.urdf (robot description, URDF)
Before this commit: robot kuka_lwr, 8 links, 7 joints
Links:
- link calib_kuka_arm_base_link: geometry collision mesh filename=meshes_kuka_lwr/convex/arm_base_convex.stl; visual mesh filename=meshes_kuka_lwr/arm_base.stl
- link kuka_arm_1_link: geometry collision mesh filename=meshes_kuka_lwr/convex/arm_segment_a_convex.stl; visual mesh filename=meshes_kuka_lwr/arm_segment_a.stl
- link kuka_arm_2_link: geometry collision mesh filename=meshes_kuka_lwr/convex/arm_segment_b_convex.stl; visual mesh filename=meshes_kuka_lwr/arm_segment_b.stl
- link kuka_arm_3_link: geometry collision mesh filename=meshes_kuka_lwr/convex/arm_segment_a_convex.stl; visual mesh filename=meshes_kuka_lwr/arm_segment_a.stl
- link kuka_arm_4_link: geometry collision mesh filename=meshes_kuka_lwr/convex/arm_segment_b_convex.stl; visual mesh filename=meshes_kuka_lwr/arm_segment_b.stl
- link kuka_arm_5_link: geometry collision mesh filename=meshes_kuka_lwr/convex/arm_segment_last_convex.stl; visual mesh filename=meshes_kuka_lwr/arm_segment_last.stl
- link kuka_arm_6_link: geometry collision mesh filename=meshes_kuka_lwr/convex/arm_wrist_convex.stl; visual mesh filename=meshes_kuka_lwr/arm_wrist.stl
- link kuka_arm_7_link: geometry collision mesh filename=meshes_kuka_lwr/convex/arm_flanche_convex.stl; visual mesh filename=meshes_kuka_lwr/arm_flanche.stl
