Commit message: Small change to the URDF example. The rotation axis of the joints should be now more readily apparent.

File: Utilities/URDF_Models/SC_3DoF.urdf (robot description, URDF)
Before this commit: robot Chaser, 5 links, 4 joints
Links:
- link Link_1: geometry visual cylinder length=0.1 radius=0.1; visual cylinder length=0.2 radius=0.05
- link Link_2: geometry visual cylinder length=0.15 radius=0.075; visual cylinder length=0.75 radius=0.05
- link Link_3: geometry visual cylinder length=0.15 radius=0.075; visual cylinder length=0.75 radius=0.05
