Commit message: Changed the location of the SPART tests and used some of the unit testing capabilities of Matlab.

File: Tests/Test_URDF/2_iiwa_base.urdf (robot description, URDF)
Before this commit: robot lbr_iiwa, 17 links, 16 joints
Links:
- link lbr_iiwa_link_0: geometry collision mesh filename=../Utilities/URDF_Models/meshes_iiwa/link_0.stl; visual mesh filename=../Utilities/URDF_Models/meshes_iiwa/link_0.stl
- link lbr_iiwa_link_0_2: geometry collision mesh filename=../Utilities/URDF_Models/meshes_iiwa/link_0.stl; visual mesh filename=../Utilities/URDF_Models/meshes_iiwa/link_0.stl
- link lbr_iiwa_link_1: geometry collision mesh filename=../Utilities/URDF_Models/meshes_iiwa/link_1.stl; visual mesh filename=../Utilities/URDF_Models/meshes_iiwa/link_1.stl
- link lbr_iiwa_link_1_2: geometry collision mesh filename=../Utilities/URDF_Models/meshes_iiwa/link_1.stl; visual mesh filename=../Utilities/URDF_Models/meshes_iiwa/link_1.stl
- link lbr_iiwa_link_2: geometry collision mesh filename=../Utilities/URDF_Models/meshes_iiwa/link_2.stl; visual mesh filename=../Utilities/URDF_Models/meshes_iiwa/link_2.stl
- link lbr_iiwa_link_2_2: geometry collision mesh filename=../Utilities/URDF_Models/meshes_iiwa/link_2.stl; visual mesh filename=../Utilities/URDF_Models/meshes_iiwa/link_2.stl
- link lbr_iiwa_link_3: geometry collision mesh filename=../Utilities/URDF_Models/meshes_iiwa/link_3.stl; visual mesh filename=../Utilities/URDF_Models/meshes_iiwa/link_3.stl
- link lbr_iiwa_link_3_2: geometry collision mesh filename=../Utilities/URDF_Models/meshes_iiwa/link_3.stl; visual mesh filename=../Utilities/URDF_Models/meshes_iiwa/link_3.stl
- link lbr_iiwa_link_4: geometry collision mesh filename=../Utilities/URDF_Models/meshes_iiwa/link_4.stl; visual mesh filename=../Utilities/URDF_Models/meshes_iiwa/link_4.stl
- link lbr_iiwa_link_4_2: geometry collision mesh filename=../Utilities/URDF_Models/meshes_iiwa/link_4.stl; visual mesh filename=../Utilities/URDF_Models/meshes_iiwa/link_4.stl
- link lbr_iiwa_link_5: geometry collision mesh filename=../Utilities/URDF_Models/meshes_iiwa/link_5.stl; visual mesh filename=../Utilities/URDF_Models/meshes_iiwa/link_5.stl
- link lbr_iiwa_link_5_2: geometry collision mesh filename=../Utilities/URDF_Models/meshes_iiwa/link_5.stl; visual mesh filename=../Utilities/URDF_Models/meshes_iiwa/link_5.stl
- link lbr_iiwa_link_6: geometry collision mesh filename=../Utilities/URDF_Models/meshes_iiwa/link_6.stl; visual mesh filename=../Utilities/URDF_Models/meshes_iiwa/link_6.stl
- link lbr_iiwa_link_6_2: geometry collision mesh filename=../Utilities/URDF_Models/meshes_iiwa/link_6.stl; visual mesh filename=../Utilities/URDF_Models/meshes_iiwa/link_6.stl
- link lbr_iiwa_link_7: geometry collision mesh filename=../Utilities/URDF_Models/meshes_iiwa/link_7.stl; visual mesh filename=../Utilities/URDF_Models/meshes_iiwa/link_7.stl
- link lbr_iiwa_link_7_2: geometry collision mesh filename=../Utilities/URDF_Models/meshes_iiwa/link_7.stl; visual mesh filename=../Utilities/URDF_Models/meshes_iiwa/link_7.stl
