Commit message: Added end-effector as a separate link.

File: URDF_models/SC_3DoF.urdf (robot description, URDF)
Before this commit: robot Chaser, 5 links, 4 joints
Links:
- added link Link_EE, mass 0; visual sphere radius=0.1
- link Link_3: geometry visual cylinder length=0.15 radius=0.075; visual cylinder length=0.75 radius=0.05
Joints:
- added joint Joint_EE: type fixed, parent Link_3, child Link_EE, origin xyz=0 0 0.75 rpy=0 0 0, axis 1 0 0
