Commit message: Changed dimensions of the spacecraft.

File: URDF_models/Simple_Spacecraft.urdf (robot description, URDF)
Before this commit: robot Chaser, 4 links, 3 joints
Links:
- link Left_Panel: geometry visual box size=0.25 3 1.5
- link Right_Panel: geometry visual box size=0.25 3 1.5
- link Spacecraft: geometry visual box size=1.25 1.5 2
Joints:
- joint Spacecraft_Fixture: origin xyz=0 0 -0.8 rpy=0 0 0 -> xyz=0 0 1 rpy=0 0 0
- joint Spacecraft_Left_Panel: origin xyz=0 -0.5 0 rpy=0 0 0 -> xyz=0 -0.75 0 rpy=0 0 0
- joint Spacecraft_Right_Panel: origin xyz=0 0.5 0 rpy=0 0 0 -> xyz=0 0.75 0 rpy=0 0 0
